Commit message: New Update upto realsense part

File: igus_robot/urdf/igus_robot.urdf (robot description, URDF)
Before this commit: robot asm_1, 8 links, 7 joints
Links:
- added link h1_link; collision mesh filename=package://igus_robot/meshes/tool2.stl; visual mesh filename=package://igus_robot/meshes/tool2.stl
Joints:
- added joint h1_joint: type fixed, parent world, child h1_link, origin xyz=0.74603 -0.19055 0.11719 rpy=0 0 0
