Commit message: report
1.The Gazebo & Rviz is functioning without any problem.

2.The Realsense camera d435 also functioning good .

3. The PointCloud 2  has be issue the code has functioning good but the frame has some error occurs the depth point can be display.

File: rldp5_description/urdf/rldp5.urdf.xacro (robot description, xacro)
@@ -146,5 +146,5 @@
       <origin xyz="0 0 0" rpy="0 3.13 0"/>
       <geometry>
-	<mesh filename="package://rldp5_description/mesh/tool1.STL"/>
+	<mesh filename="package://rldp5_description/mesh/tool1.stl"/>
      </geometry>
      </visual>
@@ -152,5 +152,5 @@
       <origin xyz="0 0 0" rpy="0 3.13 0"/>
       <geometry>
-	<mesh filename="package://rldp5_description/mesh/tool1.STL"/>
+	<mesh filename="package://rldp5_description/mesh/tool1.stl"/>
       </geometry>
     </collision>
@@ -238,5 +238,5 @@
     <gazebo>
         <plugin name="gazebo_ros_control" filename="libgazebo_ros_control.so">
-            <robotNamespace>/rldp5</robotNamespace>
+            <robotNamespace></robotNamespace>
             <robotSimType>gazebo_ros_control/DefaultRobotHWSim</robotSimType>
             <legacyModeNS>true</legacyModeNS>
