Commit message: New Changes

File: rl_dp_5/rldp5_description/urdf/rldp5.urdf.xacro (robot description, xacro)
@@ -1,168 +1,230 @@
 <?xml version="1.0" ?>
-<robot xmlns:xacro="http://www.ros.org/wiki/xacro"
-       name="igus_robolink_rl_dp_5" >
-    <link name="world"/>
+<!-- =================================================================================== -->
+<!-- |    This document was autogenerated by xacro from /home/karthik/igus_ws/src/Moveit_Igus_RL_DP5/rl_dp_5/rldp5_description/urdf/rldp5.urdf.xacro | -->
+<!-- |    EDITING THIS FILE BY HAND IS NOT RECOMMENDED                                 | -->
+<!-- =================================================================================== -->
+<robot name="igus_robolink_rl_dp_5">
+    <link name="world" />
     <link name="base_link">
-      <visual>
-        <geometry>
-          <mesh filename="package://rldp5_description/mesh/Joint0.dae"/>
-        </geometry>
-      </visual>
-      <collision>
-        <geometry>
-          <mesh filename="package://rldp5_description/mesh/Joint0Coll.dae"/>
-        </geometry>
-      </collision>
-      <inertial>
-        <mass value="1.0"/>
-        <inertia ixx="1.0" ixy="0.0" ixz="0.0" iyy="1.0" iyz="0.0" izz="1.0"/>
-      </inertial>
-    </link>
-	<joint name="virtual_joint" type="fixed">
-	<parent link="world"/>
-	<child link="base_link"/>
-	<origin xyz="0 0 0" rpy="0 0 0"/>
-	</joint>
+        <visual>
+            <geometry>
+                <mesh filename="package://rldp5_description/mesh/Joint0.dae" />
+            </geometry>
+        </visual>
+        <collision>
+            <geometry>
+                <mesh filename="package://rldp5_description/mesh/Joint0Coll.dae" />
+            </geometry>
+        </collision>
+        <inertial>
+            <mass value="1.0" />
+            <inertia ixx="1.0" ixy="0.0" ixz="0.0" iyy="1.0" iyz="0.0" izz="1.0" />
+            <origin xyz="0 0 0" rpy="0 0 0" />
+        </inertial>
+    </link>
+    <joint name="virtual_joint" type="fixed">
+        <parent link="world" />
+        <child link="base_link" />
+        <origin rpy="0 0 0" xyz="0 0 0" />
+    </joint>
     <joint name="joint_1" type="revolute">
-      <parent link="base_link"/>
-      <child link="link_1"/>
-      <origin rpy="0.0 0.0 0.0" xyz="0.0 0 0.0095"/>
-      <axis xyz="0 0 -1"/>
-      <limit effort="330.0" lower="${-pi*7/9}" upper="${pi*7/9}" velocity="2.16"/>
+        <parent link="base_link" />
+        <child link="link_1" />
+        <origin rpy="0.0 0.0 0.0" xyz="0.0 0 0.0095" />
+        <axis xyz="0 0 -1" />
+        <limit effort="330.0" lower="-2.443460952792061" upper="2.443460952792061" velocity="2.16" />
     </joint>
     <link name="link_1">
-      <visual>
-        <geometry>
-          <mesh filename="package://rldp5_description/mesh/Joint1.dae"/>
-        </geometry>
-        <origin rpy="0 0 0" xyz="0 0 0"/>
-      </visual>
-      <collision>
-        <geometry>
-          <mesh filename="package://rldp5_description/mesh/Joint1Coll.dae"/>
-        </geometry>
-        <origin rpy="0 0 0" xyz="0 0 0"/>
-      </collision>
-      <inertial>
-        <mass value="0.1"/>
-        <inertia ixx="0.03" ixy="0.0" ixz="0.0" iyy="0.03" iyz="0.0" izz="0.03"/>
-      </inertial>
+        <visual>
+            <geometry>
+                <mesh filename="package://rldp5_description/mesh/Joint1.dae" />
+            </geometry>
+            <origin rpy="0 0 0" xyz="0 0 0" />
+        </visual>
+        <collision>
+            <geometry>
+                <mesh filename="package://rldp5_description/mesh/Joint1Coll.dae" />
+            </geometry>
+            <origin rpy="0 0 0" xyz="0 0 0" />
+        </collision>
+        <inertial>
+            <mass value="0.1" />
+            <inertia ixx="0.03" ixy="0.0" ixz="0.0" iyy="0.03" iyz="0.0" izz="0.03" />
+            <origin xyz="0 0 0" rpy="0 0 0" />
+        </inertial>
     </link>
     <joint name="joint_2" type="revolute">
-      <parent link="link_1"/>
-      <child link="link_2"/>
-      <origin rpy="0.0 0.0 0.0" xyz="0.0 0 0.145"/>
-      <axis xyz="0 1 0"/>
-      <limit effort="330.0" lower="${-pi*5/18}" upper="${pi/2}" velocity="2.16"/>
+        <parent link="link_1" />
+        <child link="link_2" />
+        <origin rpy="0.0 0.0 0.0" xyz="0.0 0 0.145" />
+        <axis xyz="0 1 0" />
+        <limit effort="330.0" lower="-0.8726646259971648" upper="1.5707963267948966" velocity="2.16" />
     </joint>
     <link name="link_2">
-      <visual>
-        <geometry>
-          <mesh filename="package://rldp5_description/mesh/Joint2.dae"/>
-        </geometry>
-        <origin rpy="0 0 0" xyz="0 0 0"/>
-      </visual>
-      <collision>
-        <geometry>
-          <mesh filename="package://rldp5_description/mesh/Joint2Coll.dae"/>
-        </geometry>
-        <origin rpy="0 0 0" xyz="0 0 0"/>
-      </collision>
-      <inertial>
-        <mass value="0.1"/>
-        <inertia ixx="0.03" ixy="0.0" ixz="0.0" iyy="0.03" iyz="0.0" izz="0.03"/>
-      </inertial>
+        <visual>
+            <geometry>
+                <mesh filename="package://rldp5_description/mesh/Joint2.dae" />
+            </geometry>
+            <origin rpy="0 0 0" xyz="0 0 0" />
+        </visual>
+        <collision>
+            <geometry>
+                <mesh filename="package://rldp5_description/mesh/Joint2Coll.dae" />
+            </geometry>
+            <origin rpy="0 0 0" xyz="0 0 0" />
+        </collision>
+        <inertial>
+            <mass value="0.1" />
+            <inertia ixx="0.03" ixy="0.0" ixz="0.0" iyy="0.03" iyz="0.0" izz="0.03" />
+            <origin xyz="0 0 0" rpy="0 0 0" />
+        </inertial>
     </link>
     <joint name="joint_3" type="revolute">
-      <parent link="link_2"/>
-      <child link="link_5"/>
-      <origin rpy="0.0 0 0.0" xyz="0.0 0.0 0.350"/>
-      <axis xyz="0 1 0"/>
-      <limit effort="330.0" lower="${-pi*41/36}" upper="${pi*5/36}" velocity="2.16"/>
+        <parent link="link_2" />
+        <child link="link_5" />
+        <origin rpy="0.0 0 0.0" xyz="0.0 0.0 0.350" />
+        <axis xyz="0 1 0" />
+        <limit effort="330.0" lower="-3.577924966588375" upper="0.4363323129985824" velocity="2.16" />
     </joint>
     <link name="link_5">
-      <visual>
-        <geometry>
-          <mesh filename="package://rldp5_description/mesh/Joint3.dae"/>
-        </geometry>
-        <origin rpy="0 0 0" xyz="0 0 0"/>
-      </visual>
-      <collision>
-        <geometry>
-          <mesh filename="package://rldp5_description/mesh/Joint3Coll.dae"/>
-        </geometry>
-        <origin rpy="0 0 0" xyz="0 0 0"/>
-      </collision>
-      <inertial>
-        <mass value="0.1"/>
-        <inertia ixx="0.03" ixy="0.0" ixz="0.0" iyy="0.03" iyz="0.0" izz="0.03"/>
-      </inertial>
+        <visual>
+            <geometry>
+                <mesh filename="package://rldp5_description/mesh/Joint3.dae" />
+            </geometry>
+            <origin rpy="0 0 0" xyz="0 0 0" />
+        </visual>
+        <collision>
+            <geometry>
+                <mesh filename="package://rldp5_description/mesh/Joint3Coll.dae" />
+            </geometry>
+            <origin rpy="0 0 0" xyz="0 0 0" />
+        </collision>
+        <inertial>
+            <mass value="0.1" />
+            <inertia ixx="0.03" ixy="0.0" ixz="0.0" iyy="0.03" iyz="0.0" izz="0.03" />
+            <origin xyz="0 0 0" rpy="0 0 0" />
+        </inertial>
     </link>
     <joint name="joint_4" type="revolute">
-      <parent link="link_5"/>
-      <child link="link_6"/>
-      <origin rpy="0.0 0.0 0.0" xyz="0.0 0 0.270"/>
-      <axis xyz="0 1 0"/>
-      <limit effort="330.0" lower="${-pi*5/9}" upper="${pi*5/9}" velocity="2.16"/>
+        <parent link="link_5" />
+        <child link="link_6" />
+        <origin rpy="0.0 0.0 0.0" xyz="0.0 0 0.270" />
+        <axis xyz="0 1 0" />
+        <limit effort="330.0" lower="-1.7453292519943295" upper="1.7453292519943295" velocity="2.16" />
     </joint>
     <link name="link_6">
-      <visual>
-        <geometry>
-          <mesh filename="package://rldp5_description/mesh/Joint4.dae"/>
-        </geometry>
-        <origin rpy="0 0 0" xyz="0 0 0"/>
-      </visual>
-      <collision>
-        <geometry>
-          <mesh filename="package://rldp5_description/mesh/Joint4Coll.dae"/>
-        </geometry>
-        <origin rpy="0 0 0" xyz="0 0 0"/>
-      </collision>
-      <inertial>
-        <mass value="0.1"/>
-        <inertia ixx="0.03" ixy="0.0" ixz="0.0" iyy="0.03" iyz="0.0" izz="0.03"/>
-      </inertial>
-    </link>
-      <joint name="joint_5" type="revolute">
-        <parent link="link_6"/>
-        <child link="link_7"/>
-        <origin rpy="0.0 0.0 0.0" xyz="0.0 0 0.1785"/>
-        <axis xyz="0 0 1"/>
-        <limit effort="330.0" lower="${-pi*179/180}" upper="${pi*179/180}" velocity="2.16"/>
-      </joint>
+        <visual>
+            <geometry>
+                <mesh filename="package://rldp5_description/mesh/Joint4.dae" />
+            </geometry>
+            <origin rpy="0 0 0" xyz="0 0 0" />
+        </visual>
+        <collision>
+            <geometry>
+                <mesh filename="package://rldp5_description/mesh/Joint4Coll.dae" />
+            </geometry>
+            <origin rpy="0 0 0" xyz="0 0 0" />
+        </collision>
+        <inertial>
+            <mass value="0.1" />
+            <inertia ixx="0.03" ixy="0.0" ixz="0.0" iyy="0.03" iyz="0.0" izz="0.03" />
+            <origin xyz="0 0 0" rpy="0 0 0" />
+        </inertial>
+    </link>
+    <joint name="joint_5" type="revolute">
+        <parent link="link_6" />
+        <child link="link_7" />
+        <origin rpy="0.0 0.0 0.0" xyz="0.0 0 0.1785" />
+        <axis xyz="0 0 1" />
+        <limit effort="330.0" lower="-3.12413936106985" upper="3.12413936106985" velocity="2.16" />
+    </joint>
     <link name="link_7">
-      <visual>
-        <geometry>
-          <mesh filename="package://rldp5_description/mesh/Joint5.dae"/>
-        </geometry>
-        <origin rpy="0 0 0" xyz="0 0 0"/>
-      </visual>
-      <collision>
-        <geometry>
-          <mesh filename="package://rldp5_description/mesh/Joint5Coll.dae"/>
-        </geometry>
-        <origin rpy="0 0 0" xyz="0 0 0"/>
-      </collision>
-      <inertial>
-        <mass value="0.1"/>
-        <inertia ixx="0.03" ixy="0.0" ixz="0.0" iyy="0.03" iyz="0.0" izz="0.03"/>
-      </inertial>
+        <visual>
+            <geometry>
+                <mesh filename="package://rldp5_description/mesh/Joint5.dae" />
+            </geometry>
+            <origin rpy="0 0 0" xyz="0 0 0" />
+        </visual>
+        <collision>
+            <geometry>
+                <mesh filename="package://rldp5_description/mesh/Joint5Coll.dae" />
+            </geometry>
+            <origin rpy="0 0 0" xyz="0 0 0" />
+        </collision>
+        <inertial>
+            <mass value="0.1" />
+            <inertia ixx="0.03" ixy="0.0" ixz="0.0" iyy="0.03" iyz="0.0" izz="0.03" />
+            <origin xyz="0 0 0" rpy="0 0 0" />
+        </inertial>
     </link>
     <joint name="joint6" type="fixed">
-      <parent link="link_7"/>
-      <child link="flange"/>
-      <origin rpy="0.0 ${-pi/2} 0.0" xyz="0.0 0 0.0115"/>
-      <axis xyz="0 0 1"/>
-      <limit effort="330.0" lower="-1.65806" upper="1.65806" velocity="2.16"/>
-    </joint>
-    <link name="flange">
-    </link>
+        <parent link="link_7" />
+        <child link="flange" />
+        <origin rpy="0.0 -1.5707963267948966 0.0" xyz="0.0 0 0.0115" />
+        <axis xyz="0 0 1" />
+        <limit effort="330.0" lower="-1.65806" upper="1.65806" velocity="2.16" />
+    </joint>
+    <link name="flange" />
     <joint name="flange_to_tool0" type="fixed">
-      <parent link="flange"/>
-      <child link="tool0"/>
-      <origin rpy="0.0 0.0 0.0" xyz="0.0 0.0 0.0"/>
-      <axis xyz="0 0 0"/>
-    </joint>
-    <link name="tool0">
-    </link>
+        <parent link="flange" />
+        <child link="tool0" />
+        <origin rpy="0.0 0.0 0.0" xyz="0.0 0.0 0.0" />
+        <axis xyz="0 0 0" />
+    </joint>
+    <link name="tool0" />
+    <transmission name="trans_joint_1">
+        <type>transmission_interface/SimpleTransmission</type>
+        <joint name="joint_1">
+            <hardwareInterface>hardware_interface/PositionJointInterface</hardwareInterface>
+        </joint>
+        <actuator name="joint_1_motor">
+            <hardwareInterface>hardware_interface/PositionJointInterface</hardwareInterface>
+            <mechanicalReduction>1</mechanicalReduction>
+        </actuator>
+    </transmission>
+    <transmission name="trans_joint_2">
+        <type>transmission_interface/SimpleTransmission</type>
+        <joint name="joint_2">
+            <hardwareInterface>hardware_interface/PositionJointInterface</hardwareInterface>
+        </joint>
+        <actuator name="joint_2_motor">
+            <hardwareInterface>hardware_interface/PositionJointInterface</hardwareInterface>
+            <mechanicalReduction>1</mechanicalReduction>
+        </actuator>
+    </transmission>
+    <transmission name="trans_joint_3">
+        <type>transmission_interface/SimpleTransmission</type>
+        <joint name="joint_3">
+            <hardwareInterface>hardware_interface/PositionJointInterface</hardwareInterface>
+        </joint>
+        <actuator name="joint_3_motor">
+            <hardwareInterface>hardware_interface/PositionJointInterface</hardwareInterface>
+            <mechanicalReduction>1</mechanicalReduction>
+        </actuator>
+    </transmission>
+    <transmission name="trans_joint_4">
+        <type>transmission_interface/SimpleTransmission</type>
+        <joint name="joint_4">
+            <hardwareInterface>hardware_interface/PositionJointInterface</hardwareInterface>
+        </joint>
+        <actuator name="joint_4_motor">
+            <hardwareInterface>hardware_interface/PositionJointInterface</hardwareInterface>
+            <mechanicalReduction>1</mechanicalReduction>
+        </actuator>
+    </transmission>
+    <transmission name="trans_joint_5">
+        <type>transmission_interface/SimpleTransmission</type>
+        <joint name="joint_5">
+            <hardwareInterface>hardware_interface/PositionJointInterface</hardwareInterface>
+        </joint>
+        <actuator name="joint_5_motor">
+            <hardwareInterface>hardware_interface/PositionJointInterface</hardwareInterface>
+            <mechanicalReduction>1</mechanicalReduction>
+        </actuator>
+    </transmission>
+    <gazebo>
+        <plugin name="gazebo_ros_control">
+            <robotNamespace>/</robotNamespace>
+        </plugin>
+    </gazebo>
 </robot>

Commit message: Changes for new code without gui

File: rl_dp_5/rldp5_description/urdf/rldp5.urdf.xacro (robot description, xacro)
@@ -59,5 +59,5 @@
         <origin rpy="0.0 0.0 0.0" xyz="0.0 0 0.145" />
         <axis xyz="0 1 0" />
-        <limit effort="330.0" lower="-0.8726646259971648" upper="1.5707963267948966" velocity="2.16" />
+        <limit effort="330.0" lower="-1.74533" upper="0.872665" velocity="2.16" />
     </joint>
     <link name="link_2">
@@ -85,5 +85,5 @@
         <origin rpy="0.0 0 0.0" xyz="0.0 0.0 0.350" />
         <axis xyz="0 1 0" />
-        <limit effort="330.0" lower="-3.577924966588375" upper="0.4363323129985824" velocity="2.16" />
+        <limit effort="330.0" lower="-2.007129" upper="2.00713" velocity="2.16" />
     </joint>
     <link name="link_5">

Commit message: Changed the URDF w.r.t joint angles

File: rl_dp_5/rldp5_description/urdf/rldp5.urdf.xacro (robot description, xacro)
@@ -59,5 +59,5 @@
         <origin rpy="0.0 0.0 0.0" xyz="0.0 0 0.145" />
         <axis xyz="0 1 0" />
-        <limit effort="330.0" lower="-0.8726646259971648" upper="1.5707963267948966" velocity="2.16" />
+        <limit effort="330.0" lower="-1.74533" upper="0.872665" velocity="2.16" />
     </joint>
     <link name="link_2">
@@ -85,5 +85,5 @@
         <origin rpy="0.0 0 0.0" xyz="0.0 0.0 0.350" />
         <axis xyz="0 1 0" />
-        <limit effort="330.0" lower="-3.577924966588375" upper="0.4363323129985824" velocity="2.16" />
+        <limit effort="330.0" lower="-2.00713" upper="2.00713" velocity="2.16" />
     </joint>
     <link name="link_5">

Commit message: Now URDF and real robot have same joint directions
Now URDF and real robot have same joint directions, so we should be able to test it on a real robot.

File: rl_dp_5/rldp5_description/urdf/rldp5.urdf.xacro (robot description, xacro)
@@ -58,5 +58,5 @@
         <child link="link_2" />
         <origin rpy="0.0 0.0 0.0" xyz="0.0 0 0.145" />
-        <axis xyz="0 1 0" />
+        <axis xyz="0 -1 0" />
         <limit effort="330.0" lower="-1.74533" upper="0.872665" velocity="2.16" />
     </joint>
@@ -84,5 +84,5 @@
         <child link="link_5" />
         <origin rpy="0.0 0 0.0" xyz="0.0 0.0 0.350" />
-        <axis xyz="0 1 0" />
+        <axis xyz="0 -1 0" />
         <limit effort="330.0" lower="-2.00713" upper="2.00713" velocity="2.16" />
     </joint>
@@ -110,5 +110,5 @@
         <child link="link_6" />
         <origin rpy="0.0 0.0 0.0" xyz="0.0 0 0.270" />
-        <axis xyz="0 1 0" />
+        <axis xyz="0 -1 0" />
         <limit effort="330.0" lower="-1.7453292519943295" upper="1.7453292519943295" velocity="2.16" />
     </joint>

Commit message: Update rldp5.urdf.xacro

File: rl_dp_5/rldp5_description/urdf/rldp5.urdf.xacro (robot description, xacro)
@@ -58,5 +58,5 @@
         <child link="link_2" />
         <origin rpy="0.0 0.0 0.0" xyz="0.0 0 0.145" />
-        <axis xyz="0 1 0" />
+        <axis xyz="0 -1 0" />
         <limit effort="330.0" lower="-1.74533" upper="0.872665" velocity="2.16" />
     </joint>
@@ -84,6 +84,6 @@
         <child link="link_5" />
         <origin rpy="0.0 0 0.0" xyz="0.0 0.0 0.350" />
-        <axis xyz="0 1 0" />
-        <limit effort="330.0" lower="-2.007129" upper="2.00713" velocity="2.16" />
+        <axis xyz="0 -1 0" />
+        <limit effort="330.0" lower="-2.00713" upper="2.00713" velocity="2.16" />
     </joint>
     <link name="link_5">
@@ -110,5 +110,5 @@
         <child link="link_6" />
         <origin rpy="0.0 0.0 0.0" xyz="0.0 0 0.270" />
-        <axis xyz="0 1 0" />
+        <axis xyz="0 -1 0" />
         <limit effort="330.0" lower="-1.7453292519943295" upper="1.7453292519943295" velocity="2.16" />
     </joint>
